File: ATmega128RFA1-dev.sch (EAGLE design)
At the start: 44 parts, among them J1 POWER_JACKSMD, J2 AVR_SPI_PRG_6PTH, Q1 16MHz, Q2 32.768kHz, U1 ATMEGA128RFA1, U2 V_REG_LDOSMD, Y1 ANTENNA2SMD5

Commit message: Rearranged CC message so more of the board fits on my display
Parts:
- removed U$1: CREATIVE_COMMONS, SparkFun:CREATIVE_COMMONS
Changed lines of the file:
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@@
 <part name="P+7" library="SparkFun" deviceset="3.3V" device=""/>
 <part name="GND22" library="SparkFun" deviceset="GND" device=""/>
-<part name="U$1" library="SparkFun" deviceset="CREATIVE_COMMONS" device=""/>
 <part name="SJ1" library="jumper" deviceset="SJ" device=""/>
 <part name="GND23" library="SparkFun" deviceset="GND" device=""/>
@@
 <instance part="P+7" gate="G$1" x="198.12" y="63.5"/>
 <instance part="GND22" gate="1" x="198.12" y="45.72"/>
-<instance part="U$1" gate="G$1" x="2.54" y="175.26"/>
 <instance part="SJ1" gate="1" x="157.48" y="45.72"/>
 <instance part="GND23" gate="1" x="152.4" y="40.64"/>
